Commit message: Ajuste1

File: urdf/r2d2_sensor.urdf (robot description, URDF)
Before this commit: robot r2d2_sensor, 15 links, 14 joints
Links:
- link box: mass 0.05 -> 0.001; geometry 
- link camera_rgb_link: mass 0.01 -> 0.001; geometry 
- link lidar3d_link: mass 0.02 -> 0.001; geometry 

Commit message: Ajuste2

File: urdf/r2d2_sensor.urdf (robot description, URDF)
Before this commit: robot r2d2_sensor, 15 links, 14 joints
Links:
- link box: geometry visual box size=0.08 0.2 0.1
